Commit message: Add files via upload

File: Model/wheel.xacro (robot description, xacro)
@@ -7,4 +7,5 @@
       <link name="body${pos}">
       <collision>
+         <origin xyz="0 0 0" rpy="${roll} ${pit} ${yaw}"/>
           <geometry>
             <mesh filename="package://urdf_tutorial/Wheel2_Double_ohneRaeder.stl" scale=".0021 .0021 .0021"/>
@@ -21,21 +22,34 @@
 <inertia ixx="0.00236" ixy ="0" ixz="0" iyy="0.00236" iyz="0" izz="0.00945"/>
 </inertial>
+<gazebo>
+<gravity> 1 </gravity>
+<dampingFactor>10</dampingFactor>
+<mu1>0.6</mu1>
+<mu2>0.6</mu2>
+</gazebo>
       </link>
      <link name="roller1${pos}">
        <collision >
-          <geometry>
-            <mesh filename="package://urdf_tutorial/Wheel2_wheel_rightOrient.stl" scale=".0021 .0021 .0021"/>
-          </geometry>
-        </collision>
-        <visual >
            <origin xyz="0 0 0" rpy="0 0 1.57079"/>
-           <geometry>
-            <mesh filename="package://urdf_tutorial/Wheel2_wheel_rightOrient.stl" scale=".0021 .0021 .0021"/>
-          </geometry>
-        </visual>
-<inertial>
-         <mass value = "0.05"/>
-<inertia ixx="0.000018" ixy ="0" ixz="0" iyy="0.00000722" iyz="0.0" izz="0.00000722"/>
-</inertial>
+          <geometry>
+            <mesh filename="package://urdf_tutorial/Wheel2_wheel_rightOrient.stl" scale=".0021 .0021 .0021"/>
+          </geometry>
+        </collision>
+        <visual >
+           <origin xyz="0 0 0" rpy="0 0 1.57079"/>
+           <geometry>
+            <mesh filename="package://urdf_tutorial/Wheel2_wheel_rightOrient.stl" scale=".0021 .0021 .0021"/>
+          </geometry>
+        </visual>
+<inertial>
+         <mass value = "0.05"/>
+<inertia ixx="0.000018" ixy ="0" ixz="0" iyy="0.00000722" iyz="0.0" izz="0.00000722"/>
+</inertial>
+<gazebo>
+<gravity> 1 </gravity>
+<dampingFactor>10</dampingFactor>
+<mu1>0.6</mu1>
+<mu2>0.6</mu2>
+</gazebo>
       </link>
     <joint name="1${pos}" type="continuous">
@@ -47,18 +61,25 @@
     <link name="roller2${pos}">
        <collision >
-          <geometry>
-            <mesh filename="package://urdf_tutorial/Wheel2_wheel_rightOrient.stl" scale=".0021 .0021 .0021"/>
-          </geometry>
-        </collision>
-        <visual >
            <origin xyz="0 0 0" rpy="0 -1.25664 1.57079"/>
-           <geometry>
-            <mesh filename="package://urdf_tutorial/Wheel2_wheel_rightOrient.stl" scale=".0021 .0021 .0021"/>
-          </geometry>
-        </visual>
-<inertial>
-         <mass value = "0.05"/>
-<inertia ixx="0.000018" ixy ="0" ixz="0" iyy="0.00000722" iyz="0.0" izz="0.00000722"/>
-</inertial>
+          <geometry>
+            <mesh filename="package://urdf_tutorial/Wheel2_wheel_rightOrient.stl" scale=".0021 .0021 .0021"/>
+          </geometry>
+        </collision>
+        <visual >
+           <origin xyz="0 0 0" rpy="0 -1.25664 1.57079"/>
+           <geometry>
+            <mesh filename="package://urdf_tutorial/Wheel2_wheel_rightOrient.stl" scale=".0021 .0021 .0021"/>
+          </geometry>
+        </visual>
+<inertial>
+         <mass value = "0.05"/>
+<inertia ixx="0.000018" ixy ="0" ixz="0" iyy="0.00000722" iyz="0.0" izz="0.00000722"/>
+</inertial>
+<gazebo>
+<gravity> 1 </gravity>
+<dampingFactor>10</dampingFactor>
+<mu1>0.6</mu1>
+<mu2>0.6</mu2>
+</gazebo>
       </link>
     <joint name="2${pos}" type="continuous">
@@ -70,18 +91,25 @@
      <link name="roller3${pos}">
         <collision >
-          <geometry>
-            <mesh filename="package://urdf_tutorial/Wheel2_wheel_rightOrient.stl" scale=".0021 .0021 .0021"/>
-          </geometry>
-        </collision>
-        <visual >
            <origin xyz="0 0 0" rpy="0 -2.5132 1.57079"/>
-           <geometry>
-            <mesh filename="package://urdf_tutorial/Wheel2_wheel_rightOrient.stl" scale=".0021 .0021 .0021"/>
-          </geometry>
-        </visual>
-<inertial>
-         <mass value = "0.05"/>
-<inertia ixx="0.000018" ixy ="0" ixz="0" iyy="0.00000722" iyz="0.0" izz="0.00000722"/>
-</inertial>
+          <geometry>
+            <mesh filename="package://urdf_tutorial/Wheel2_wheel_rightOrient.stl" scale=".0021 .0021 .0021"/>
+          </geometry>
+        </collision>
+        <visual >
+           <origin xyz="0 0 0" rpy="0 -2.5132 1.57079"/>
+           <geometry>
+            <mesh filename="package://urdf_tutorial/Wheel2_wheel_rightOrient.stl" scale=".0021 .0021 .0021"/>
+          </geometry>
+        </visual>
+<inertial>
+         <mass value = "0.05"/>
+<inertia ixx="0.000018" ixy ="0" ixz="0" iyy="0.00000722" iyz="0.0" izz="0.00000722"/>
+</inertial>
+<gazebo>
+<gravity> 1 </gravity>
+<dampingFactor>10</dampingFactor>
+<mu1>0.6</mu1>
+<mu2>0.6</mu2>
+</gazebo>
       </link>
     <joint name="3${pos}" type="continuous">
@@ -93,18 +121,25 @@
      <link name="roller4${pos}">
            <collision >
-          <geometry>
-            <mesh filename="package://urdf_tutorial/Wheel2_wheel_rightOrient.stl" scale=".0021 .0021 .0021"/>
-          </geometry>
-        </collision>
-        <visual >
            <origin xyz="0 0 0" rpy="0 -3.7699 1.57079"/>
-           <geometry>
-            <mesh filename="package://urdf_tutorial/Wheel2_wheel_rightOrient.stl" scale=".0021 .0021 .0021"/>
-          </geometry>
-        </visual>
-<inertial>
-         <mass value = "0.05"/>
-<inertia ixx="0.000018" ixy ="0" ixz="0" iyy="0.00000722" iyz="0.0" izz="0.00000722"/>
-</inertial>
+          <geometry>
+            <mesh filename="package://urdf_tutorial/Wheel2_wheel_rightOrient.stl" scale=".0021 .0021 .0021"/>
+          </geometry>
+        </collision>
+        <visual >
+           <origin xyz="0 0 0" rpy="0 -3.7699 1.57079"/>
+           <geometry>
+            <mesh filename="package://urdf_tutorial/Wheel2_wheel_rightOrient.stl" scale=".0021 .0021 .0021"/>
+          </geometry>
+        </visual>
+<inertial>
+         <mass value = "0.05"/>
+<inertia ixx="0.000018" ixy ="0" ixz="0" iyy="0.00000722" iyz="0.0" izz="0.00000722"/>
+</inertial>
+<gazebo>
+<gravity> 1 </gravity>
+<dampingFactor>10</dampingFactor>
+<mu1>0.6</mu1>
+<mu2>0.6</mu2>
+</gazebo>
       </link>
     <joint name="4${pos}" type="continuous">
@@ -116,18 +151,25 @@
      <link name="roller5${pos}">
         <collision >
-          <geometry>
-            <mesh filename="package://urdf_tutorial/Wheel2_wheel_rightOrient.stl" scale=".0021 .0021 .0021"/>
-          </geometry>
-        </collision>
-        <visual >
            <origin xyz="0 0 0" rpy="0 1.25664 1.57079"/>
-           <geometry>
-            <mesh filename="package://urdf_tutorial/Wheel2_wheel_rightOrient.stl" scale=".0021 .0021 .0021"/>
-          </geometry>
-        </visual>
-<inertial>
-         <mass value = "0.05"/>
-<inertia ixx="0.000018" ixy ="0" ixz="0" iyy="0.00000722" iyz="0.0" izz="0.00000722"/>
-</inertial>
+          <geometry>
+            <mesh filename="package://urdf_tutorial/Wheel2_wheel_rightOrient.stl" scale=".0021 .0021 .0021"/>
+          </geometry>
+        </collision>
+        <visual >
+           <origin xyz="0 0 0" rpy="0 1.25664 1.57079"/>
+           <geometry>
+            <mesh filename="package://urdf_tutorial/Wheel2_wheel_rightOrient.stl" scale=".0021 .0021 .0021"/>
+          </geometry>
+        </visual>
+<inertial>
+         <mass value = "0.05"/>
+<inertia ixx="0.000018" ixy ="0" ixz="0" iyy="0.00000722" iyz="0.0" izz="0.00000722"/>
+</inertial>
+<gazebo>
+<gravity> 1 </gravity>
+<dampingFactor>10</dampingFactor>
+<mu1>0.6</mu1>
+<mu2>0.6</mu2>
+</gazebo>
       </link>
     <joint name="5${pos}" type="continuous">
@@ -139,18 +181,25 @@
      <link name="roller6${pos}">
        <collision >
-          <geometry>
-            <mesh filename="package://urdf_tutorial/Wheel2_wheel_rightOrient.stl" scale=".0021 .0021 .0021"/>
-          </geometry>
-        </collision>
-        <visual >
            <origin xyz="0 0 0" rpy="0 -0.6283 1.57079"/>
-           <geometry>
-            <mesh filename="package://urdf_tutorial/Wheel2_wheel_rightOrient.stl" scale=".0021 .0021 .0021"/>
-          </geometry>
-        </visual>
-<inertial>
-         <mass value = "0.05"/>
-<inertia ixx="0.000018" ixy ="0" ixz="0" iyy="0.00000722" iyz="0.0" izz="0.00000722"/>
-</inertial>
+          <geometry>
+            <mesh filename="package://urdf_tutorial/Wheel2_wheel_rightOrient.stl" scale=".0021 .0021 .0021"/>
+          </geometry>
+        </collision>
+        <visual >
+           <origin xyz="0 0 0" rpy="0 -0.6283 1.57079"/>
+           <geometry>
+            <mesh filename="package://urdf_tutorial/Wheel2_wheel_rightOrient.stl" scale=".0021 .0021 .0021"/>
+          </geometry>
+        </visual>
+<inertial>
+         <mass value = "0.05"/>
+<inertia ixx="0.000018" ixy ="0" ixz="0" iyy="0.00000722" iyz="0.0" izz="0.00000722"/>
+</inertial>
+<gazebo>
+<gravity> 1 </gravity>
+<dampingFactor>10</dampingFactor>
+<mu1>0.6</mu1>
+<mu2>0.6</mu2>
+</gazebo>
       </link>
     <joint name="6${pos}" type="continuous">
@@ -162,18 +211,25 @@
      <link name="roller7${pos}">
       <collision >
-          <geometry>
-            <mesh filename="package://urdf_tutorial/Wheel2_wheel_rightOrient.stl" scale=".0021 .0021 .0021"/>
-          </geometry>
-        </collision>
-        <visual >
            <origin xyz="0 0 0" rpy="0 -1.8849 1.57079"/>
-           <geometry>
-            <mesh filename="package://urdf_tutorial/Wheel2_wheel_rightOrient.stl" scale=".0021 .0021 .0021"/>
-          </geometry>
-        </visual>
-<inertial>
-         <mass value = "0.05"/>
-<inertia ixx="0.000018" ixy ="0" ixz="0" iyy="0.00000722" iyz="0.0" izz="0.00000722"/>
-</inertial>
+          <geometry>
+            <mesh filename="package://urdf_tutorial/Wheel2_wheel_rightOrient.stl" scale=".0021 .0021 .0021"/>
+          </geometry>
+        </collision>
+        <visual >
+           <origin xyz="0 0 0" rpy="0 -1.8849 1.57079"/>
+           <geometry>
+            <mesh filename="package://urdf_tutorial/Wheel2_wheel_rightOrient.stl" scale=".0021 .0021 .0021"/>
+          </geometry>
+        </visual>
+<inertial>
+         <mass value = "0.05"/>
+<inertia ixx="0.000018" ixy ="0" ixz="0" iyy="0.00000722" iyz="0.0" izz="0.00000722"/>
+</inertial>
+<gazebo>
+<gravity> 1 </gravity>
+<dampingFactor>10</dampingFactor>
+<mu1>0.6</mu1>
+<mu2>0.6</mu2>
+</gazebo>
       </link>
     <joint name="7${pos}" type="continuous">
@@ -185,18 +241,25 @@
      <link name="roller8${pos}">
       <collision >
-          <geometry>
-            <mesh filename="package://urdf_tutorial/Wheel2_wheel_rightOrient.stl" scale=".0021 .0021 .0021"/>
-          </geometry>
-        </collision>
-        <visual >
            <origin xyz="0 0 0" rpy="0 -3.14159 1.57079"/>
-           <geometry>
-            <mesh filename="package://urdf_tutorial/Wheel2_wheel_rightOrient.stl" scale=".0021 .0021 .0021"/>
-          </geometry>
-        </visual>
-<inertial>
-         <mass value = "0.05"/>
-<inertia ixx="0.000018" ixy ="0" ixz="0" iyy="0.00000722" iyz="0.0" izz="0.00000722"/>
-</inertial>
+          <geometry>
+            <mesh filename="package://urdf_tutorial/Wheel2_wheel_rightOrient.stl" scale=".0021 .0021 .0021"/>
+          </geometry>
+        </collision>
+        <visual >
+           <origin xyz="0 0 0" rpy="0 -3.14159 1.57079"/>
+           <geometry>
+            <mesh filename="package://urdf_tutorial/Wheel2_wheel_rightOrient.stl" scale=".0021 .0021 .0021"/>
+          </geometry>
+        </visual>
+<inertial>
+         <mass value = "0.05"/>
+<inertia ixx="0.000018" ixy ="0" ixz="0" iyy="0.00000722" iyz="0.0" izz="0.00000722"/>
+</inertial>
+<gazebo>
+<gravity> 1 </gravity>
+<dampingFactor>10</dampingFactor>
+<mu1>0.6</mu1>
+<mu2>0.6</mu2>
+</gazebo>
       </link>
     <joint name="8${pos}" type="continuous">
@@ -208,18 +271,25 @@
      <link name="roller9${pos}">
       <collision >
-          <geometry>
-            <mesh filename="package://urdf_tutorial/Wheel2_wheel_rightOrient.stl" scale=".0021 .0021 .0021"/>
-          </geometry>
-        </collision>
-        <visual >
            <origin xyz="0 0 0" rpy="0 -4.3982 1.57079"/>
-           <geometry>
-            <mesh filename="package://urdf_tutorial/Wheel2_wheel_rightOrient.stl" scale=".0021 .0021 .0021"/>
-          </geometry>
-        </visual>
-<inertial>
-         <mass value = "0.05"/>
-<inertia ixx="0.000018" ixy ="0" ixz="0" iyy="0.00000722" iyz="0.0" izz="0.00000722"/>
-</inertial>
+          <geometry>
+            <mesh filename="package://urdf_tutorial/Wheel2_wheel_rightOrient.stl" scale=".0021 .0021 .0021"/>
+          </geometry>
+        </collision>
+        <visual >
+           <origin xyz="0 0 0" rpy="0 -4.3982 1.57079"/>
+           <geometry>
+            <mesh filename="package://urdf_tutorial/Wheel2_wheel_rightOrient.stl" scale=".0021 .0021 .0021"/>
+          </geometry>
+        </visual>
+<inertial>
+         <mass value = "0.05"/>
+<inertia ixx="0.000018" ixy ="0" ixz="0" iyy="0.00000722" iyz="0.0" izz="0.00000722"/>
+</inertial>
+<gazebo>
+<gravity> 1 </gravity>
+<dampingFactor>10</dampingFactor>
+<mu1>0.6</mu1>
+<mu2>0.6</mu2>
+</gazebo>
       </link>
     <joint name="9${pos}" type="continuous">
@@ -231,18 +301,25 @@
      <link name="roller10${pos}">
        <collision >
-          <geometry>
-            <mesh filename="package://urdf_tutorial/Wheel2_wheel_rightOrient.stl" scale=".0021 .0021 .0021"/>
-          </geometry>
-        </collision>
-        <visual >
            <origin xyz="0 0 0" rpy="0 -5.6548 1.57079"/>
-           <geometry>
-            <mesh filename="package://urdf_tutorial/Wheel2_wheel_rightOrient.stl" scale=".0021 .0021 .0021"/>
-          </geometry>
-        </visual>
-<inertial>
-         <mass value = "0.05"/>
-<inertia ixx="0.000018" ixy ="0" ixz="0" iyy="0.00000722" iyz="0.0" izz="0.00000722"/>
-</inertial>
+          <geometry>
+            <mesh filename="package://urdf_tutorial/Wheel2_wheel_rightOrient.stl" scale=".0021 .0021 .0021"/>
+          </geometry>
+        </collision>
+        <visual >
+           <origin xyz="0 0 0" rpy="0 -5.6548 1.57079"/>
+           <geometry>
+            <mesh filename="package://urdf_tutorial/Wheel2_wheel_rightOrient.stl" scale=".0021 .0021 .0021"/>
+          </geometry>
+        </visual>
+<inertial>
+         <mass value = "0.05"/>
+<inertia ixx="0.000018" ixy ="0" ixz="0" iyy="0.00000722" iyz="0.0" izz="0.00000722"/>
+</inertial>
+<gazebo>
+<gravity> 1 </gravity>
+<dampingFactor>10</dampingFactor>
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